Commit message: Update package references to 'bme_gazebo_sensors1' in launch and URDF files

File: bme_gazebo_sensors1/urdf/mogi_bot.urdf (robot description, URDF)
Before this commit: robot mogi_bot, 5 links, 4 joints
Links:
- link base_link: geometry collision box size=.4 .2 .1; collision sphere radius=0.0499
- link left_wheel: geometry collision cylinder length=.05 radius=.1; visual mesh filename=package://bme_gazebo_sensors1/meshes/wheel.dae
- link right_wheel: geometry collision cylinder length=.05 radius=.1; visual mesh filename=package://bme_gazebo_sensors1/meshes/wheel.dae
- link scan_link: geometry collision box size=.1 .1 .1; visual mesh filename=package://bme_gazebo_sensors1/meshes/lidar.dae
